Commit message: Model gripper pads with compliant hydroelastic boxes

File: movo_common/movo_description/urdf/manipulation/robotiq/robotiq_85_gripper.urdf (robot description, URDF)
Before this commit: robot robotiq85_gripper, 10 links, 9 joints
Links:
- link gripper_finger1_finger_tip_link: geometry collision box size=0.054846 0.022487 0.022000; visual mesh filename=package://movo_description/meshes/manipulation/robotiq/visu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
- link gripper_finger2_finger_tip_link: geometry collision box size=0.054846 0.022487 0.022000; visual mesh filename=package://movo_description/meshes/manipulation/robotiq/visu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
